File: ESP-LIS3DH/esp-lis3dh.brd (EAGLE design)
At the start: 46 x 30 mm, 22 parts, among them IC2 4043PW, IC3 CP2104-F03-GM, IC4 MCP73831/OT, U1 LIS3DHTR, U4 SN74LVC1G04

Commit message: Worked on pcb
Parts:
- added LED2: RED, microbuilder:CHIPLED_0805
- added LED3: ORANGE, microbuilder:CHIPLED_0805
- added R10: 500k, microbuilder:0603
- added R7, R8: 1k, microbuilder:0603
- added R9: 100k, microbuilder:0603
- added SW1: SPST_TACT-KMR2, adafruit:KMR2
- LED1: value ORANGE -> GREEN
- moved C1 1.00 mm to (18.0, 19.0)
- moved R1 1.00 mm to (14.0, 19.0)
- moved R5 1.00 mm to (20.0, 19.0)
- moved R6 1.00 mm to (16.0, 19.0)
Connections:
- new net ADC: R10.1, R9.1, X1.2
- new net GPIO12: R8.1, X1.6
- new net GPIO13: R7.1, X1.7
- new net GPIO15: R5.2, SW1.3, X1.10
- new net N$7: LED3.A, R8.2
- net GND: now also LED2.C, LED3.C, R10.2
- net N$3: now also LED2.A, R7.2; no longer R5.2, X1.10
- net VCC: now also R9.2, SW1.4
Routing:
- net GPIO12: track 0.00 -> 31.3 mm, vias 0 -> 2
- net GPIO13: track 0.00 -> 30.2 mm, vias 0 -> 2
- net VCC: track 48.1 -> 76.8 mm
- net ADC: track 0.00 -> 23.1 mm, vias 0 -> 2
- net GPIO15: track 0.00 -> 9.22 mm
- net N$3: track 6.89 -> 2.08 mm
- net N$7: track 0.00 -> 2.10 mm
- net EN: track 44.0 -> 45.3 mm
- net DTR: track 38.5 -> 39.7 mm
- net N$2: track 4.90 -> 5.90 mm
- net 5.0V: track 29.4 -> 30.2 mm
- net N$4: track 6.00 -> 5.41 mm
- net GND: vias 15 -> 19

Commit message: Worked on prototype
Parts:
- added PAD1, PAD2: (no value), wirepad:SMD1,27-2,54
- added U$7, U$8: MOUNTINGHOLE2.5, microbuilder:MOUNTINGHOLE_2.5_PLATED
- moved R8 9.43 mm to (14.0, 2.00), turned to 180 degrees
- moved LED3 4.47 mm to (10.0, 5.00), turned to 0 degrees
- moved C1 2.00 mm to (18.0, 21.0)
- moved R1 2.00 mm to (14.0, 21.0)
- moved R6 2.00 mm to (16.0, 21.0)
- moved C2 1.00 mm to (12.1, 24.8)
- moved LED1 1.00 mm to (7.00, 27.0)
- moved R4 1.00 mm to (9.00, 27.0)
Connections:
- new net BATLOW: IC2.9, R8.1
- new net GPIO14: IC2.7, X1.5
- net GND: now also PAD2.1; no longer U1.10
- net GPIO12: now also IC2.6; no longer R8.1
- net VBAT: now also PAD1.1
Routing:
- net GPIO14: track 0.00 -> 27.4 mm, vias 0 -> 2
- net GND: track 11.7 -> 3.47 mm, vias 19 -> 31
- net GPIO12: track 31.3 -> 23.8 mm
- net VCC: track 76.8 -> 82.5 mm
- net DTR: track 39.7 -> 35.7 mm
- net VBAT: track 6.78 -> 9.69 mm
- net BATLOW: track 0.00 -> 2.67 mm
- net N$4: track 5.41 -> 2.94 mm
- net N$2: track 5.90 -> 7.90 mm
- net RXD: track 32.3 -> 34.3 mm
- net N$7: track 2.10 -> 3.96 mm
- net N$1: track 8.63 -> 10.4 mm, vias 0 -> 2
- net SETLATCH: track 34.2 -> 35.9 mm, vias 3 -> 2
- net N$10: track 20.2 -> 18.6 mm
- net N$9: track 4.61 -> 5.85 mm
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