File: ESP-LIS3DH/esp-lis3dh.sch (EAGLE design)
At the start: 22 parts, among them IC2 4043PW, IC3 CP2104-F03-GM, IC4 MCP73831/OT, U1 LIS3DHTR, U4 SN74LVC1G04

Commit message: Worked on pcb
Parts:
- added LED2: RED, microbuilder:LED0805
- added LED3: ORANGE, microbuilder:LED0805
- added R10: 500k, microbuilder:RESISTOR0603
- added R7, R8: 1k, microbuilder:RESISTOR0603
- added R9: 100k, microbuilder:RESISTOR0603
- added SW1: SPST_TACT-KMR2, adafruit:SPST_TACT-KMR2
- LED1: value ORANGE -> GREEN
Connections:
- new net ADC: R10.1, R9.1, X1.ADC
- new net GPIO12: R8.1, X1.GPIO12
- new net GPIO13: R7.1, X1.GPIO13
- new net GPIO15: R5.2, SW1.P1, X1.GPIO15
- new net N$7: LED3.A, R8.2
- net GND: now also LED2.C, LED3.C, R10.2
- net N$3: now also LED2.A, R7.2; no longer R5.2, X1.GPIO15
- net VCC: now also R9.2, SW1.S1
Changed lines of the file:
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@@
 <part name="U$4" library="microbuilder" deviceset="5.0V" device=""/>
 <part name="U$5" library="microbuilder" deviceset="VBAT" device=""/>
-<part name="LED1" library="microbuilder" deviceset="LED" device="0805" value="ORANGE"/>
+<part name="LED1" library="microbuilder" deviceset="LED" device="0805" value="GREEN"/>
 <part name="R4" library="microbuilder" deviceset="RESISTOR" device="0603" value="1k"/>
 <part name="R6" library="microbuilder" deviceset="RESISTOR" device="0603" value="1k"/>
@@
 <part name="IC2" library="masterthesis" deviceset="4043" device="PW"/>
 <part name="U$6" library="microusb" deviceset="MICRO-USB" device=""/>
+<part name="R7" library="microbuilder" deviceset="RESISTOR" device="0603" value="1k"/>
+<part name="R8" library="microbuilder" deviceset="RESISTOR" device="0603" value="1k"/>
+<part name="GND10" library="supply1" library_urn="urn:adsk.eagle:library:371" deviceset="GND" device=""/>
+<part name="GND11" library="supply1" library_urn="urn:adsk.eagle:library:371" deviceset="GND" device=""/>
+<part name="LED2" library="microbuilder" deviceset="LED" device="0805" value="RED"/>
+<part name="LED3" library="microbuilder" deviceset="LED" device="0805" value="ORANGE"/>
+<part name="P+4" library="supply1" library_urn="urn:adsk.eagle:library:371" deviceset="VCC" device=""/>
+<part name="GND12" library="supply1" library_urn="urn:adsk.eagle:library:371" deviceset="GND" device=""/>
+<part name="R9" library="microbuilder" deviceset="RESISTOR" device="0603" value="100k"/>
+<part name="R10" library="microbuilder" deviceset="RESISTOR" device="0603" value="500k"/>
+<part name="SW1" library="adafruit" library_urn="urn:adsk.eagle:library:420" deviceset="SPST_TACT" device="-KMR2"/>
+<part name="P+8" library="supply1" library_urn="urn:adsk.eagle:library:371" deviceset="VCC" device=""/>
 </parts>
 <sheets>
@@
 <instance part="IC2" gate="A" x="-45.72" y="88.9" rot="R270"/>
 <instance part="U$6" gate="G$1" x="-144.78" y="111.76"/>
+<instance part="R7" gate="G$1" x="58.42" y="58.42" rot="R90"/>
+<instance part="R8" gate="G$1" x="68.58" y="58.42" rot="R90"/>
+<instance part="GND10" gate="1" x="58.42" y="73.66" rot="R180"/>
+<instance part="GND11" gate="1" x="68.58" y="73.66" rot="R180"/>
+<instance part="LED2" gate="G$1" x="58.42" y="68.58" rot="R90"/>
+<instance part="LED3" gate="G$1" x="68.58" y="68.58" rot="R90"/>
+<instance part="P+4" gate="VCC" x="58.42" y="114.3"/>
+<instance part="GND12" gate="1" x="68.58" y="114.3" rot="R180"/>
+<instance part="R9" gate="G$1" x="58.42" y="106.68" rot="R90"/>
+<instance part="R10" gate="G$1" x="68.58" y="106.68" rot="R90"/>
+<instance part="SW1" gate="G$1" x="83.82" y="58.42"/>
+<instance part="P+8" gate="VCC" x="86.36" y="66.04"/>
 </instances>
 <busses>
@@
 <pinref part="U$6" gate="G$1" pin="GND"/>
 </segment>
+<segment>
+<pinref part="LED2" gate="G$1" pin="C"/>
+<pinref part="GND10" gate="1" pin="GND"/>
+</segment>
+<segment>
+<pinref part="LED3" gate="G$1" pin="C"/>
+<pinref part="GND11" gate="1" pin="GND"/>
+</segment>
+<segment>
+<pinref part="GND12" gate="1" pin="GND"/>
+<pinref part="R10" gate="G$1" pin="2"/>
+</segment>
 </net>
 <net name="VCC" class="0">
@@
 <pinref part="IC2" gate="A" pin="EN"/>
 </segment>
+<segment>
+<pinref part="P+4" gate="VCC" pin="VCC"/>
+<pinref part="R9" gate="G$1" pin="2"/>
+</segment>
+<segment>
+<pinref part="SW1" gate="G$1" pin="S1"/>
+<pinref part="P+8" gate="VCC" pin="VCC"/>
+</segment>
 </net>
 <net name="EN" class="0">
@@
 </segment>
 </net>
-<net name="N$3" class="0">
+<net name="GPIO15" class="0">
 <segment>
 <pinref part="X1" gate="G$1" pin="GPIO15"/>
 <wire x1="30.48" y1="38.1" x2="35.56" y2="38.1" width="0.1524" layer="91"/>
 <pinref part="R5" gate="G$1" pin="2"/>
+<label x="30.48" y="38.1" size="1.778" layer="95"/>
+</segment>
+<segment>
+<pinref part="SW1" gate="G$1" pin="P1"/>
+<wire x1="86.36" y1="53.34" x2="86.36" y2="43.18" width="0.1524" layer="91"/>
+<label x="86.36" y="43.18" size="1.778" layer="95" rot="R90"/>
 </segment>
 </net>
@@
 <segment>
 <pinref part="X1" gate="G$1" pin="GPIO16"/>
-<label x="-12.7" y="58.42" size="1.778" layer="95" rot="R270"/>
+<label x="-12.7" y="60.96" size="1.778" layer="95" rot="R270"/>
 <wire x1="-5.08" y1="45.72" x2="-10.16" y2="45.72" width="0.1524" layer="91"/>
 <wire x1="-10.16" y1="45.72" x2="-10.16" y2="55.88" width="0.1524" layer="91"/>
@@
 </segment>
 </net>
+<net name="GPIO13" class="0">
+<segment>
+<pinref part="X1" gate="G$1" pin="GPIO13"/>
+<wire x1="-5.08" y1="38.1" x2="-15.24" y2="38.1" width="0.1524" layer="91"/>
+<label x="-15.24" y="38.1" size="1.778" layer="95"/>
+</segment>
+<segment>
+<pinref part="R7" gate="G$1" pin="1"/>
+<wire x1="58.42" y1="53.34" x2="58.42" y2="43.18" width="0.1524" layer="91"/>
+<label x="58.42" y="43.18" size="1.778" layer="95" rot="R90"/>
+</segment>
+</net>
+<net name="GPIO12" class="0">
+<segment>
+<pinref part="X1" gate="G$1" pin="GPIO12"/>
+<wire x1="-5.08" y1="40.64" x2="-15.24" y2="40.64" width="0.1524" layer="91"/>
+<label x="-15.24" y="40.64" size="1.778" layer="95"/>
+</segment>
+<segment>
+<pinref part="R8" gate="G$1" pin="1"/>
+<wire x1="68.58" y1="53.34" x2="68.58" y2="43.18" width="0.1524" layer="91"/>
+<label x="68.58" y="43.18" size="1.778" layer="95" rot="R90"/>
+</segment>
+</net>
+<net name="ADC" class="0">
+<segment>
+<pinref part="X1" gate="G$1" pin="ADC"/>
+<wire x1="-5.08" y1="50.8" x2="-7.62" y2="50.8" width="0.1524" layer="91"/>
+<wire x1="-7.62" y1="50.8" x2="-7.62" y2="63.5" width="0.1524" layer="91"/>
+<label x="-5.08" y="55.88" size="1.778" layer="95" rot="R90"/>
+</segment>
+<segment>
+<pinref part="R9" gate="G$1" pin="1"/>
+<pinref part="R10" gate="G$1" pin="1"/>
+<wire x1="58.42" y1="101.6" x2="63.5" y2="101.6" width="0.1524" layer="91"/>
+<junction x="63.5" y="101.6"/>
+<wire x1="63.5" y1="101.6" x2="68.58" y2="101.6" width="0.1524" layer="91"/>
+<wire x1="63.5" y1="101.6" x2="63.5" y2="93.98" width="0.1524" layer="91"/>
+<label x="63.5" y="93.98" size="1.778" layer="95" rot="R90"/>
+</segment>
+</net>
+<net name="N$3" class="0">
+<segment>
+<pinref part="R7" gate="G$1" pin="2"/>
+<pinref part="LED2" gate="G$1" pin="A"/>
+</segment>
+</net>
+<net name="N$7" class="0">
+<segment>
+<pinref part="R8" gate="G$1" pin="2"/>
+<pinref part="LED3" gate="G$1" pin="A"/>
+</segment>
+</net>

Commit message: Worked on prototype
Parts:
- added PAD1, PAD2: (no value), wirepad:SMD2
- added U$7, U$8: MOUNTINGHOLE2.5, microbuilder:MOUNTINGHOLE2.5
Connections:
- new net BATLOW: IC2A.Q1, R8.1
- new net GPIO14: IC2A.R1, X1.GPIO14
- net GND: now also PAD2.P, U$6.GND@1, U$6.GND@2; no longer U1.RES(GND)
- net GPIO12: now also IC2A.S1; no longer R8.1
- net VBAT: now also PAD1.P
Other:
- moved on the sheet: U4
Changed lines of the file:
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@@
 <?xml version="1.0" encoding="utf-8"?>
 <!DOCTYPE eagle SYSTEM "eagle.dtd">
-<eagle version="8.3.2">
+<eagle version="8.4.1">
 <drawing>
 <settings>
@@
 <part name="X1" library="adafruit" deviceset="ESP-12" device=""/>
 <part name="U1" library="microbuilder" deviceset="ACCEL_LIS3DHTR" device="" value="LIS3DHTR"/>
-<part name="GND1" library="supply1" library_urn="urn:adsk.eagle:library:371" deviceset="GND" device=""/>
 <part name="GND2" library="supply1" library_urn="urn:adsk.eagle:library:371" deviceset="GND" device=""/>
 <part name="P+1" library="supply1" library_urn="urn:adsk.eagle:library:371" deviceset="VCC" device=""/>
 <part name="P+2" library="supply1" library_urn="urn:adsk.eagle:library:371" deviceset="VCC" device=""/>
-<part name="GND3" library="supply1" library_urn="urn:adsk.eagle:library:371" deviceset="GND" device=""/>
-<part name="GND4" library="supply1" library_urn="urn:adsk.eagle:library:371" deviceset="GND" device=""/>
 <part name="P+3" library="supply1" library_urn="urn:adsk.eagle:library:371" deviceset="VCC" device=""/>
 <part name="P+5" library="supply1" library_urn="urn:adsk.eagle:library:371" deviceset="VCC" device=""/>
@@
 <part name="SW1" library="adafruit" library_urn="urn:adsk.eagle:library:420" deviceset="SPST_TACT" device="-KMR2"/>
 <part name="P+8" library="supply1" library_urn="urn:adsk.eagle:library:371" deviceset="VCC" device=""/>
+<part name="U$7" library="microbuilder" deviceset="MOUNTINGHOLE" device="2.5"/>
+<part name="U$8" library="microbuilder" deviceset="MOUNTINGHOLE" device="2.5"/>
+<part name="PAD1" library="wirepad" library_urn="urn:adsk.eagle:library:412" deviceset="SMD2" device="" package3d_urn="urn:adsk.eagle:package:30839/1"/>
+<part name="PAD2" library="wirepad" library_urn="urn:adsk.eagle:library:412" deviceset="SMD2" device="" package3d_urn="urn:adsk.eagle:package:30839/1"/>
+<part name="GND13" library="supply1" library_urn="urn:adsk.eagle:library:371" deviceset="GND" device=""/>
+<part name="U$9" library="microbuilder" deviceset="VBAT" device=""/>
+<part name="GND14" library="supply1" library_urn="urn:adsk.eagle:library:371" deviceset="GND" device=""/>
+<part name="GND15" library="supply1" library_urn="urn:adsk.eagle:library:371" deviceset="GND" device=""/>
+<part name="GND1" library="supply1" library_urn="urn:adsk.eagle:library:371" deviceset="GND" device=""/>
+<part name="GND3" library="supply1" library_urn="urn:adsk.eagle:library:371" deviceset="GND" device=""/>
 </parts>
 <sheets>
 <sheet>
 <plain>
-<frame x1="-142.24" y1="17.78" x2="104.14" y2="134.62" columns="8" rows="5" layer="91"/>
+<frame x1="-149.86" y1="17.78" x2="96.52" y2="134.62" columns="8" rows="5" layer="91"/>
 <wire x1="-71.12" y1="129.54" x2="-71.12" y2="76.2" width="0.1524" layer="94"/>
 <wire x1="-71.12" y1="76.2" x2="-71.12" y2="22.86" width="0.1524" layer="94"/>
@@
 <instance part="X1" gate="G$1" x="12.7" y="48.26"/>
 <instance part="U1" gate="G$1" x="-48.26" y="55.88"/>
-<instance part="GND1" gate="1" x="-30.48" y="58.42" rot="R90"/>
 <instance part="GND2" gate="1" x="27.94" y="27.94" rot="R270"/>
 <instance part="P+1" gate="VCC" x="-7.62" y="35.56" rot="R90"/>
 <instance part="P+2" gate="VCC" x="-45.72" y="73.66"/>
-<instance part="GND3" gate="1" x="-66.04" y="50.8" rot="R270"/>
-<instance part="GND4" gate="1" x="-30.48" y="53.34" rot="R90"/>
 <instance part="P+3" gate="VCC" x="-66.04" y="60.96" rot="R90"/>
 <instance part="P+5" gate="VCC" x="-60.96" y="104.14"/>
@@
 <instance part="C2" gate="G$1" x="27.94" y="91.44" rot="R90"/>
 <instance part="C3" gate="G$1" x="-12.7" y="109.22"/>
-<instance part="U4" gate="G$1" x="-38.1" y="116.84"/>
-<instance part="P+7" gate="VCC" x="-40.64" y="127"/>
-<instance part="GND5" gate="1" x="-40.64" y="106.68"/>
+<instance part="U4" gate="G$1" x="-43.18" y="116.84"/>
+<instance part="P+7" gate="VCC" x="-45.72" y="127"/>
+<instance part="GND5" gate="1" x="-45.72" y="106.68"/>
 <instance part="IC2" gate="A" x="-45.72" y="88.9" rot="R270"/>
 <instance part="U$6" gate="G$1" x="-144.78" y="111.76"/>
@@
 <instance part="SW1" gate="G$1" x="83.82" y="58.42"/>
 <instance part="P+8" gate="VCC" x="86.36" y="66.04"/>
+<instance part="U$7" gate="G$1" x="83.82" y="119.38"/>
+<instance part="U$8" gate="G$1" x="83.82" y="111.76"/>
+<instance part="PAD1" gate="1" x="30.48" y="109.22"/>
+<instance part="PAD2" gate="1" x="30.48" y="101.6"/>
+<instance part="GND13" gate="1" x="35.56" y="101.6" rot="R90"/>
+<instance part="U$9" gate="G$1" x="35.56" y="109.22" rot="R270"/>
+<instance part="GND14" gate="1" x="-139.7" y="91.44"/>
+<instance part="GND15" gate="1" x="-142.24" y="91.44"/>
+<instance part="GND1" gate="1" x="-66.04" y="50.8" rot="R270"/>
+<instance part="GND3" gate="1" x="-30.48" y="58.42" rot="R90"/>
 </instances>
 <busses>
@@
 <nets>
 <net name="GND" class="0">
-<segment>
-<pinref part="U1" gate="G$1" pin="RES(GND)"/>
-<pinref part="GND4" gate="1" pin="GND"/>
-</segment>
-<segment>
-<pinref part="U1" gate="G$1" pin="GND@2"/>
-<pinref part="GND1" gate="1" pin="GND"/>
-</segment>
 <segment>
 <pinref part="X1" gate="G$1" pin="GND"/>
@@
 <pinref part="R5" gate="G$1" pin="1"/>
 <wire x1="35.56" y1="27.94" x2="30.48" y2="27.94" width="0.1524" layer="91"/>
-</segment>
-<segment>
-<pinref part="U1" gate="G$1" pin="GND@1"/>
-<pinref part="GND3" gate="1" pin="GND"/>
 </segment>
 <segment>
@@
 <pinref part="GND12" gate="1" pin="GND"/>
 <pinref part="R10" gate="G$1" pin="2"/>
+</segment>
+<segment>
+<pinref part="PAD2" gate="1" pin="P"/>
+<pinref part="GND13" gate="1" pin="GND"/>
+</segment>
+<segment>
+<pinref part="U$6" gate="G$1" pin="GND@2"/>
+<pinref part="GND14" gate="1" pin="GND"/>
+</segment>
+<segment>
+<pinref part="U$6" gate="G$1" pin="GND@1"/>
+<pinref part="GND15" gate="1" pin="GND"/>
+</segment>
+<segment>
+<pinref part="U1" gate="G$1" pin="GND@1"/>
+<pinref part="GND1" gate="1" pin="GND"/>
+</segment>
+<segment>
+<pinref part="U1" gate="G$1" pin="GND@2"/>
+<pinref part="GND3" gate="1" pin="GND"/>
 </segment>
 </net>
@@
 </segment>
 <segment>
-<wire x1="-48.26" y1="116.84" x2="-60.96" y2="116.84" width="0.1524" layer="91"/>
-<label x="-63.5" y="116.84" size="1.778" layer="95"/>
+<wire x1="-53.34" y1="116.84" x2="-66.04" y2="116.84" width="0.1524" layer="91"/>
+<label x="-68.58" y="116.84" size="1.778" layer="95"/>
 <pinref part="U4" gate="G$1" pin="A"/>
 </segment>
@@
 <wire x1="20.32" y1="91.44" x2="22.86" y2="91.44" width="0.1524" layer="91"/>
 </segment>
+<segment>
+<pinref part="PAD1" gate="1" pin="P"/>
+<pinref part="U$9" gate="G$1" pin="VBAT"/>
+</segment>
 </net>
 <net name="N$4" class="0">
@@
 </segment>
 </net>
-<net name="N$1" class="0">
-<segment>
-<pinref part="U4" gate="G$1" pin="Y"/>
-<wire x1="-33.02" y1="116.84" x2="-33.02" y2="101.6" width="0.1524" layer="91"/>
-<pinref part="IC2" gate="A" pin="R0"/>
-</segment>
-</net>
 <net name="GPIO13" class="0">
 <segment>
@@
 </segment>
 <segment>
-<pinref part="R8" gate="G$1" pin="1"/>
-<wire x1="68.58" y1="53.34" x2="68.58" y2="43.18" width="0.1524" layer="91"/>
-<label x="68.58" y="43.18" size="1.778" layer="95" rot="R90"/>
+<pinref part="IC2" gate="A" pin="S1"/>
+<wire x1="-38.1" y1="101.6" x2="-38.1" y2="106.68" width="0.1524" layer="91"/>
+<label x="-35.56" y="101.6" size="1.778" layer="95" rot="R90"/>
 </segment>
 </net>
@@
 </segment>
 </net>
+<net name="BATLOW" class="0">
+<segment>
+<pinref part="IC2" gate="A" pin="Q1"/>
+<wire x1="-38.1" y1="76.2" x2="-38.1" y2="73.66" width="0.1524" layer="91"/>
+<label x="-38.1" y="78.74" size="1.778" layer="95" rot="R270"/>
+</segment>
+<segment>
+<pinref part="R8" gate="G$1" pin="1"/>
+<wire x1="68.58" y1="53.34" x2="68.58" y2="43.18" width="0.1524" layer="91"/>
+<label x="68.58" y="43.18" size="1.778" layer="95" rot="R90"/>
+</segment>
+</net>
+<net name="N$1" class="0">
+<segment>
+<pinref part="U4" gate="G$1" pin="Y"/>
+<wire x1="-38.1" y1="116.84" x2="-33.02" y2="116.84" width="0.1524" layer="91"/>
+<pinref part="IC2" gate="A" pin="R0"/>
+<wire x1="-33.02" y1="116.84" x2="-33.02" y2="101.6" width="0.1524" layer="91"/>
+</segment>
+</net>
+<net name="GPIO14" class="0">
+<segment>
+<pinref part="IC2" gate="A" pin="R1"/>
+<wire x1="-40.64" y1="101.6" x2="-40.64" y2="106.68" width="0.1524" layer="91"/>
+<label x="-40.64" y="101.6" size="1.778" layer="95" rot="R90"/>
+</segment>
+<segment>
+<pinref part="X1" gate="G$1" pin="GPIO14"/>
+<wire x1="-5.08" y1="43.18" x2="-15.24" y2="43.18" width="0.1524" layer="91"/>
+<label x="-15.24" y="43.18" size="1.778" layer="95"/>
+</segment>
+</net>
