File: ESPind/espind.sch (EAGLE design)
At the start: 18 parts, among them IC1 MCP73831/OT, U2 CP2104-F03-GM, U3 AP2112-3.3

Commit message: NEW TAG PCB
Parts:
- added 3.3VPAD, 5VPAD, AC1, AC2, ADCPAD, BAT, ENPAD, GND, RESETPAD, SETPAD, VBUSPAD: (no value), wirepad:SMD2
- added C10: 4.7uF, microbuilder:CAP_CERAMIC0603
- added C11, C6, C7: 22nF, microbuilder:CAP_CERAMIC0402
- added C12, C13: 10nF, microbuilder:CAP_CERAMIC0402
- added C5: 10uF, microbuilder:CAP_CERAMIC0402
- added C8, C9: 470nF, microbuilder:CAP_CERAMIC0402
- added LED1, LED4: GREEN, microbuilder:LED0603
- added LED2, LED5: RED, microbuilder:LED0603
- added LED3: ORANGE, microbuilder:LED0603
- added R10, R12: 100k, microbuilder:RESISTOR0402
- added R11, R7: 2k, microbuilder:RESISTOR0402
- added R13: 500k, microbuilder:RESISTOR0402
- added R14, R15, R16, R17: 1k, microbuilder:RESISTOR0402
- added R8: 10k, microbuilder:RESISTOR0402
- added R9: 140, microbuilder:RESISTOR0402
- added SW1: SPST_TACT-KMR2, adafruit:SPST_TACT-KMR2
- added U$11: BQ51013B, masterthesis:BQ51013B
- added U$12: CD4043B, masterthesis:CD4043B
- added U$30, U$31: MOUNTINGHOLE2.5, microbuilder:MOUNTINGHOLE2.5
- added U4: (no value), microbuilder:ACCEL_LIS3DHTR
- added U5: SN74LVC1G04, epic:SN74LVC1G04
- C2: value 10uF -> 10nF
- C3, C4: value 10uF -> 4.7uF; device microbuilder:CAP_CERAMIC0402 -> microbuilder:CAP_CERAMIC0603
- R6: value 10k -> 1k
Connections:
- new net $N99: C11.P$1, C3.P$2, R10.1, U$11.RECT
- new net +5V: 5VPAD.P, C4.P$1, D1.C, IC1.VDD, LED1.A, R5.1, U$11.OUT, U3.IN
- new net AC1: AC1.P, C12.P$1, C7.P$1, C9.P$1, U$11.AC1
- new net AC2: AC2.P, C13.P$2, C6.P$2, C8.P$2, U$11.AC2
- new net BATLOW: R15.1, U$12.Q2
- new net CHG: IC1.STAT, R6.2, U$11.~CHG
- new net FOD: R10.2, R11.2, R9.1, U$11.FOD
- new net GPIO15: R4.1, SW1.P1, X1.GPIO15
- new net N$10: C8.P$1, U$11.CLAMP2
- new net N$11: R11.1, U$11.ILIM
- new net N$12: C9.P$2, U$11.CLAMP1
- new net N$13: C7.P$2, U$11.COMM1
- new net N$14: C6.P$1, U$11.COMM2
- new net N$15: LED2.A, R14.2
- new net N$16: LED3.A, R15.2
- new net N$17: C12.P$2, U$11.BOOT1
- new net N$18: C13.P$1, U$11.BOOT2
- new net N$19: LED4.C, U2.GPIO0
- new net N$20: LED5.C, U2.GPIO1
- new net N$7: LED1.C, R6.1
- new net N$8: IC1.PROG, R7.2
- new net N$9: R8.1, U$11.TS/CTRL
- new net RESETLATCH: RESETPAD.P, U$12.R1, U5.Y
- new net SETLATCH: SETPAD.P, U$12.S1, U4.INT1
- new net V+: BAT.P, C5.P$1, D1.A, IC1.VBAT, R12.2
- net ADC: now also ADCPAD.P, R12.1, R13.2
- net EN: now also ENPAD.P, U$12.Q1
- net GND: now also C10.P$1, C11.P$2, C3.P$1, C4.P$2, C5.P$2, GND.P, IC1.VSS, LED2.C, LED3.C, R13.1, R7.1, R8.2, R9.2, U$11.AD, U$11.PGND, U$11.PGND2, U$11.RES, U$12.GND, U4.GND@1, U4.GND@2, U4.RES(GND), U5.GND; no longer C3.P$2, C4.P$1
- net GPIO12: now also U$12.S2
- net GPIO13: now also R14.1
- net GPIO14: now also U$12.R2
- net GPIO16: now also U5.A
- net N$2: now also LED5.A, R16.1; no longer R4.1, X1.GPIO15
- net N$6: now also LED4.A, R17.1; no longer IC1.STAT, R6.2
- net SCL: now also U4.SCL
- net SDA: now also U4.SDA
- net VBUS: now also C10.P$2, VBUSPAD.P; no longer C4.P$2
- net VCC: now also 3.3VPAD.P, R16.2, R17.2, SW1.S1, U$12.EN, U$12.VCC, U4.VDD, U4.VDDIO, U5.VCC; no longer C3.P$1, D1.A, D1.C, R5.1, U3.IN
Other:
- moved on the sheet: C3, C4, IC1, R1, R2, R3, R4, R6, T1, T2, U2
